Commit message: feat(bai03): complete Lab 3 - physical gripper, camera perception, 5 cubes and conflict resolution

File: src/ur3_llm_control/urdf/ur_with_gripper.urdf.xacro (robot description, xacro)
@@ -34,8 +34,8 @@
     <origin xyz="0 0 0" rpy="0 0 0"/>
   </joint>
-  <!-- 2. Ngón kẹp trái (Left Finger) -->
+  <!-- 2. Ngon kep trai (Left Finger - Active Prismatic Joint) -->
   <link name="gripper_left_finger">
     <visual>
-      <origin xyz="0 0.015 0.025" rpy="0 0 0"/>
+      <origin xyz="0 0 0.025" rpy="0 0 0"/>
       <geometry>
         <box size="0.016 0.008 0.05"/>
@@ -46,5 +46,5 @@
     </visual>
     <collision>
-      <origin xyz="0 0.015 0.025" rpy="0 0 0"/>
+      <origin xyz="0 0 0.025" rpy="0 0 0"/>
       <geometry>
         <box size="0.016 0.008 0.05"/>
@@ -52,18 +52,20 @@
     </collision>
     <inertial>
-      <mass value="0.03"/>
-      <origin xyz="0 0.015 0.025" rpy="0 0 0"/>
-      <inertia ixx="0.00001" ixy="0" ixz="0" iyy="0.00001" iyz="0" izz="0.00001"/>
+      <mass value="0.05"/>
+      <origin xyz="0 0 0.025" rpy="0 0 0"/>
+      <inertia ixx="0.0001" ixy="0" ixz="0" iyy="0.0001" iyz="0" izz="0.0001"/>
     </inertial>
   </link>
-  <joint name="gripper_left_joint" type="fixed">
+  <joint name="gripper_left_joint" type="prismatic">
     <parent link="gripper_base"/>
     <child link="gripper_left_finger"/>
-    <origin xyz="0 0 0.04" rpy="0 0 0"/>
+    <origin xyz="0 0.02 0.04" rpy="0 0 0"/>
+    <axis xyz="0 1 0"/>
+    <limit lower="-0.01" upper="0.025" effort="100.0" velocity="0.2"/>
   </joint>
-  <!-- 3. Ngón kẹp phải (Right Finger) -->
+  <!-- 3. Ngon kep phai (Right Finger - Active Prismatic Joint) -->
   <link name="gripper_right_finger">
     <visual>
-      <origin xyz="0 -0.015 0.025" rpy="0 0 0"/>
+      <origin xyz="0 0 0.025" rpy="0 0 0"/>
       <geometry>
         <box size="0.016 0.008 0.05"/>
@@ -74,5 +76,5 @@
     </visual>
     <collision>
-      <origin xyz="0 -0.015 0.025" rpy="0 0 0"/>
+      <origin xyz="0 0 0.025" rpy="0 0 0"/>
       <geometry>
         <box size="0.016 0.008 0.05"/>
@@ -80,15 +82,17 @@
     </collision>
     <inertial>
-      <mass value="0.03"/>
-      <origin xyz="0 -0.015 0.025" rpy="0 0 0"/>
-      <inertia ixx="0.00001" ixy="0" ixz="0" iyy="0.00001" iyz="0" izz="0.00001"/>
+      <mass value="0.05"/>
+      <origin xyz="0 0 0.025" rpy="0 0 0"/>
+      <inertia ixx="0.0001" ixy="0" ixz="0" iyy="0.0001" iyz="0" izz="0.0001"/>
     </inertial>
   </link>
-  <joint name="gripper_right_joint" type="fixed">
+  <joint name="gripper_right_joint" type="prismatic">
     <parent link="gripper_base"/>
     <child link="gripper_right_finger"/>
-    <origin xyz="0 0 0.04" rpy="0 0 0"/>
+    <origin xyz="0 -0.02 0.04" rpy="0 0 0"/>
+    <axis xyz="0 1 0"/>
+    <limit lower="-0.025" upper="0.01" effort="100.0" velocity="0.2"/>
   </joint>
-  <!-- 4. Điểm tác động kẹp trung tâm (Tool Center Point - TCP) -->
+  <!-- 4. Diem tac dong kep trung tam (Tool Center Point - TCP) -->
   <link name="gripper_tcp"/>
   <joint name="gripper_tcp_joint" type="fixed">
@@ -97,3 +101,69 @@
     <origin xyz="0 0 0.08" rpy="0 0 0"/>
   </joint>
+  <!-- GAZEBO PLUGINS: DIEU KHIEN KHOP KEP & CO CHE DONG/MO VAT THE -->
+  <gazebo>
+    <plugin
+      filename="ignition-gazebo-joint-position-controller-system"
+      name="ignition::gazebo::systems::JointPositionController">
+      <joint_name>gripper_left_joint</joint_name>
+      <topic>/gripper/left_cmd</topic>
+      <p_gain>200.0</p_gain>
+      <i_gain>1.0</i_gain>
+      <d_gain>0.5</d_gain>
+      <cmd_max>100.0</cmd_max>
+      <cmd_min>-100.0</cmd_min>
+    </plugin>
+    <plugin
+      filename="ignition-gazebo-joint-position-controller-system"
+      name="ignition::gazebo::systems::JointPositionController">
+      <joint_name>gripper_right_joint</joint_name>
+      <topic>/gripper/right_cmd</topic>
+      <p_gain>200.0</p_gain>
+      <i_gain>1.0</i_gain>
+      <d_gain>0.5</d_gain>
+      <cmd_max>100.0</cmd_max>
+      <cmd_min>-100.0</cmd_min>
+    </plugin>
+    <!-- DetachableJoint cho 5 vat the -->
+    <plugin filename="ignition-gazebo-detachable-joint-system"
+            name="ignition::gazebo::systems::DetachableJoint">
+      <parent_link>tool0</parent_link>
+      <child_model>red_cube</child_model>
+      <child_link>link</child_link>
+      <detach_topic>/gripper/detach_red</detach_topic>
+      <attach_topic>/gripper/attach_red</attach_topic>
+    </plugin>
+    <plugin filename="ignition-gazebo-detachable-joint-system"
+            name="ignition::gazebo::systems::DetachableJoint">
+      <parent_link>tool0</parent_link>
+      <child_model>yellow_cube</child_model>
+      <child_link>link</child_link>
+      <detach_topic>/gripper/detach_yellow</detach_topic>
+      <attach_topic>/gripper/attach_yellow</attach_topic>
+    </plugin>
+    <plugin filename="ignition-gazebo-detachable-joint-system"
+            name="ignition::gazebo::systems::DetachableJoint">
+      <parent_link>tool0</parent_link>
+      <child_model>blue_cube</child_model>
+      <child_link>link</child_link>
+      <detach_topic>/gripper/detach_blue</detach_topic>
+      <attach_topic>/gripper/attach_blue</attach_topic>
+    </plugin>
+    <plugin filename="ignition-gazebo-detachable-joint-system"
+            name="ignition::gazebo::systems::DetachableJoint">
+      <parent_link>tool0</parent_link>
+      <child_model>green_cube</child_model>
+      <child_link>link</child_link>
+      <detach_topic>/gripper/detach_green</detach_topic>
+      <attach_topic>/gripper/attach_green</attach_topic>
+    </plugin>
+    <plugin filename="ignition-gazebo-detachable-joint-system"
+            name="ignition::gazebo::systems::DetachableJoint">
+      <parent_link>tool0</parent_link>
+      <child_model>purple_cube</child_model>
+      <child_link>link</child_link>
+      <detach_topic>/gripper/detach_purple</detach_topic>
+      <attach_topic>/gripper/attach_purple</attach_topic>
+    </plugin>
+  </gazebo>
 </robot>

Commit message: Complete Lab 03 camera guided grasp planning

File: src/ur3_llm_control/urdf/ur_with_gripper.urdf.xacro (robot description, xacro)
@@ -110,5 +110,5 @@
       <origin xyz="0 -0.005 0.022" rpy="0 0 0"/>
       <geometry>
-        <box size="0.022 0.006 0.040"/>
+        <box size="0.028 0.006 0.040"/>
       </geometry>
     </collision>
@@ -151,5 +151,5 @@
       <origin xyz="0 0.005 0.022" rpy="0 0 0"/>
       <geometry>
-        <box size="0.022 0.006 0.040"/>
+        <box size="0.028 0.006 0.040"/>
       </geometry>
     </collision>
@@ -176,5 +176,5 @@
   </joint>
   <!-- ======================================================================= -->
-  <!-- GAZEBO SURFACE FRICTION: MA SÁT TIẾP XÚC CỰC LỚN ĐỂ GẮP VẬT THẬT         -->
+  <!-- GAZEBO SURFACE FRICTION: MA SÁT ĐỆM SILICONE VỪA PHẢI, TRÁNH TÍCH LỰC KHI NHẢ         -->
   <!-- ======================================================================= -->
   <gazebo reference="gripper_left_finger">
@@ -183,6 +183,6 @@
         <friction>
           <ode>
-            <mu>100.0</mu>
-            <mu2>100.0</mu2>
+            <mu>2.0</mu>
+            <mu2>2.0</mu2>
             <slip1>0.0</slip1>
             <slip2>0.0</slip2>
@@ -191,7 +191,7 @@
         <contact>
           <ode>
-            <kp>1000000.0</kp>
+            <kp>100000.0</kp>
             <kd>100.0</kd>
-            <min_depth>0.001</min_depth>
+            <min_depth>0.0002</min_depth>
           </ode>
         </contact>
@@ -204,6 +204,6 @@
         <friction>
           <ode>
-            <mu>100.0</mu>
-            <mu2>100.0</mu2>
+            <mu>2.0</mu>
+            <mu2>2.0</mu2>
             <slip1>0.0</slip1>
             <slip2>0.0</slip2>
@@ -212,7 +212,7 @@
         <contact>
           <ode>
-            <kp>1000000.0</kp>
+            <kp>100000.0</kp>
             <kd>100.0</kd>
-            <min_depth>0.001</min_depth>
+            <min_depth>0.0002</min_depth>
           </ode>
         </contact>

Commit message: Stabilize grasping and enforce student ID sorting

File: src/ur3_llm_control/urdf/ur_with_gripper.urdf.xacro (robot description, xacro)
@@ -107,5 +107,5 @@
     </visual>
     <!-- Mặt tiếp xúc va chạm ma sát cao -->
-    <collision>
+    <collision name="left_finger_pad_collision">
       <origin xyz="0 -0.005 0.022" rpy="0 0 0"/>
       <geometry>
@@ -148,5 +148,5 @@
     </visual>
     <!-- Mặt tiếp xúc va chạm ma sát cao -->
-    <collision>
+    <collision name="right_finger_pad_collision">
       <origin xyz="0 0.005 0.022" rpy="0 0 0"/>
       <geometry>
@@ -183,6 +183,6 @@
         <friction>
           <ode>
-            <mu>2.0</mu>
-            <mu2>2.0</mu2>
+            <mu>2.5</mu>
+            <mu2>2.5</mu2>
             <slip1>0.0</slip1>
             <slip2>0.0</slip2>
@@ -198,4 +198,15 @@
       </surface>
     </collision>
+    <sensor name="left_finger_contact_sensor" type="contact">
+      <always_on>true</always_on>
+      <update_rate>100</update_rate>
+      <contact>
+        <!-- sdformat them prefix/suffix nay khi chuyen URDF collision co ten. -->
+        <collision>gripper_left_finger_fixed_joint_lump__left_finger_pad_collision_collision</collision>
+        <!-- Gazebo Fortress doc topic o BEN TRONG contact. Dat ben ngoai lam
+             sdformat sinh __default_topic__ va ROS bridge khong nhan du lieu. -->
+        <topic>/gripper/left_contacts</topic>
+      </contact>
+    </sensor>
   </gazebo>
   <gazebo reference="gripper_right_finger">
@@ -204,6 +215,6 @@
         <friction>
           <ode>
-            <mu>2.0</mu>
-            <mu2>2.0</mu2>
+            <mu>2.5</mu>
+            <mu2>2.5</mu2>
             <slip1>0.0</slip1>
             <slip2>0.0</slip2>
@@ -219,4 +230,12 @@
       </surface>
     </collision>
+    <sensor name="right_finger_contact_sensor" type="contact">
+      <always_on>true</always_on>
+      <update_rate>100</update_rate>
+      <contact>
+        <collision>gripper_right_finger_fixed_joint_lump__right_finger_pad_collision_collision</collision>
+        <topic>/gripper/right_contacts</topic>
+      </contact>
+    </sensor>
   </gazebo>
   <!-- ======================================================================= -->
@@ -229,7 +248,7 @@
       <joint_name>gripper_left_joint</joint_name>
       <topic>/gripper/left_cmd</topic>
-      <p_gain>60.0</p_gain>
+      <p_gain>80.0</p_gain>
       <i_gain>0.1</i_gain>
-      <d_gain>5.0</d_gain>
+      <d_gain>8.0</d_gain>
       <cmd_max>25.0</cmd_max>
       <cmd_min>-25.0</cmd_min>
@@ -240,7 +259,7 @@
       <joint_name>gripper_right_joint</joint_name>
       <topic>/gripper/right_cmd</topic>
-      <p_gain>60.0</p_gain>
+      <p_gain>80.0</p_gain>
       <i_gain>0.1</i_gain>
-      <d_gain>5.0</d_gain>
+      <d_gain>8.0</d_gain>
       <cmd_max>25.0</cmd_max>
       <cmd_min>-25.0</cmd_min>
